File: 12v-front-pcb/12v-front-pcb.sch (KiCad schematic (older format))
At the start: 48 parts

Commit message: Re-work front PCB
Parts:
- removed B1, B10, B2, B3, B4, B5, B6, B7, B8, B9: 282836-6, Socket:2828366, symbol Connector:282836-6
- added COOLANT_PUMP_RELAY1, DASHBOARD_RELAY2, RADIO_RELAY1: DZ85AB-5-PCB, Socket:DZ85AB5PCB, symbol DZ85AB-5-PCB:DZ85AB-5-PCB
- added D3, D4: 10A10, Diode_THT:DIOAD1165W56L425D185, symbol Diode:10A10
- added J1: 1-776180-1, 17761801, symbol Connector:1-776180-1
- added J2: 776087-4, 7760874, symbol Connector:776087-4
- added J3: 776267-1, 776267-1, symbol Connector:776267-1
- added J4, J5: 1-776280-1, 17762801, symbol Connector:1-776280-1
- renumbered WATER_PUMP_FUSE1 to COOLANT_PUMP_FUSE1
Connections:
- net BMS_12V is gone; now on an unnamed net: BMS_RELAY1.3
- net HEADLIGHTS is gone; now on net HEADLIGHT_12V: HEADLIGHT_RELAY1.3
- net 12V_BATT: no longer BMS_FUSE1.1, BMS_FUSE1.8, DASHBOARD_FUSE1.1, DASHBOARD_FUSE1.2, DASHBOARD_FUSE1.7, DASHBOARD_FUSE1.8, FLASHER_FUSE1.1, FLASHER_FUSE1.2, FLASHER_FUSE1.7, FLASHER_FUSE1.8, INTERIOR_LIGHTS_FUSE1.1, INTERIOR_LIGHTS_FUSE1.2, INTERIOR_LIGHTS_FUSE1.7, INTERIOR_LIGHTS_FUSE1.8
- net BRAKE_SWITCH_A: now also IGNITION_RELAY1.1, D3.2, J1.11, J1.13, J1.17, J1.23, J1.5, J1.7, J1.9, J5.1, RADIO_RELAY1.4; no longer COOLANT_PUMP_FUSE1.1, COOLANT_PUMP_FUSE1.2, COOLANT_PUMP_FUSE1.7, COOLANT_PUMP_FUSE1.8, IGNITION_RELAY1.3, RADIO_FUSE1.1, RADIO_FUSE1.2, RADIO_FUSE1.7, RADIO_FUSE1.8
- net CHARGER_ON_SIGNAL: now also D4.2, DASHBOARD_RELAY2.4, J3.5
- net COOLANT_PUMP: now also COOLANT_PUMP_RELAY1.1, J2.10; no longer COOLANT_PUMP_FUSE1.3, COOLANT_PUMP_FUSE1.4, COOLANT_PUMP_FUSE1.5, COOLANT_PUMP_FUSE1.6
- net DASHBOARD_12V: now also DASHBOARD_RELAY1.1, J4.1; no longer DASHBOARD_RELAY1.3
- net DASH_HIGHBEAM_INDICATOR: now also HIGHBEAM_RELAY1.1, J2.13, J2.14, J4.4; no longer HIGHBEAM_RELAY1.3
- net DASH_INDICATOR_INDICATOR: now also J4.2
- net DRIVE_INHIBIT: now also FWD_DRIVE_INHIBIT_RELAY1.4, REV_DRIVE_INHIBIT_RELAY1.4, J3.8; no longer FWD_DRIVE_INHIBIT_RELAY1.5, REV_DRIVE_INHIBIT_RELAY1.5
- net FLASHER_B: now also LH_INDICATOR_RELAY1.3, RH_INDICATOR_RELAY1.3; no longer LH_INDICATOR_RELAY1.1, RH_INDICATOR_RELAY1.1
- net HAZARD_SWITCH_B: now also J1.2
- net HEADLIGHT_12V: no longer HEADLIGHT_RELAY1.1
- net HEADLIGHT_SWITCH_B: now also HEADLIGHT_RELAY1.4, J1.6; no longer HEADLIGHT_RELAY1.5
- net HEATER_FAN_12V: now also J2.9
- net HIGHBEAM_SWITCH_B: now also HIGHBEAM_RELAY1.4, J1.8; no longer HIGHBEAM_RELAY1.5
- net HORN: now also HORN_RELAY1.1, J2.17; no longer HORN_RELAY1.3
- net HORN_SWITCH_B: now also HORN_RELAY1.4, J1.18; no longer HORN_RELAY1.5
- net HVJB_12V: now also J2.18
- net IGNITION_SWITCH_B: now also IGNITION_RELAY1.4, J1.4; no longer IGNITION_RELAY1.5
- net INTERIOR_LIGHTS: now also INTERIOR_LIGHTS_RELAY1.1, J1.20; no longer INTERIOR_LIGHTS_RELAY1.3
- net INTERIOR_LIGHT_SWITCH_B: now also INTERIOR_LIGHTS_RELAY1.4, J1.16; no longer INTERIOR_LIGHTS_RELAY1.5
- net INVERTER_12V: now also J2.3
- net INVERTER_FWD: now also J2.6
- net INVERTER_REV: now also J2.7, J3.7
- net LH_INDICATOR_SWITCH_B: now also J1.10
- net RADIO_12V: now also J1.22, RADIO_RELAY1.1; no longer RADIO_FUSE1.3, RADIO_FUSE1.4, RADIO_FUSE1.5, RADIO_FUSE1.6
- net RH_INDICATOR_SWITCH_B: now also J1.12
- net SHIFTER_FWD: now also FWD_DRIVE_INHIBIT_RELAY1.3, J5.3; no longer FWD_DRIVE_INHIBIT_RELAY1.1
- net SHIFTER_REV: now also REV_DRIVE_INHIBIT_RELAY1.3, J5.2; no longer REV_DRIVE_INHIBIT_RELAY1.1
- net VACUUM_PUMP: now also J2.8
- net IGNITION_SWITCH_A: now reaches IGNITION_FUSE1.3, IGNITION_FUSE1.4, IGNITION_FUSE1.5, IGNITION_FUSE1.6
- net IGNITION_SWITCH_A: now also COOLANT_PUMP_FUSE1.1, COOLANT_PUMP_FUSE1.2, COOLANT_PUMP_FUSE1.7, COOLANT_PUMP_FUSE1.8, IGNITION_RELAY1.3, INTERIOR_LIGHTS_FUSE1.1, INTERIOR_LIGHTS_FUSE1.2, INTERIOR_LIGHTS_FUSE1.7, INTERIOR_LIGHTS_FUSE1.8, RADIO_FUSE1.1, RADIO_FUSE1.2, RADIO_FUSE1.7, RADIO_FUSE1.8, J1.15, J1.3, J3.14; no longer IGNITION_RELAY1.1
- net at D11.1, D12.1: now also LH_INDICATOR_RELAY1.4; no longer LH_INDICATOR_RELAY1.5
- net at D13.1, D14.1: now also RH_INDICATOR_RELAY1.4; no longer RH_INDICATOR_RELAY1.5
- net at HEADLIGHT_FUSE1.3, HEADLIGHT_FUSE1.4, HEADLIGHT_FUSE1.5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: now also HIGHBEAM_RELAY1.3; no longer HIGHBEAM_RELAY1.1
- net at INTERIOR_LIGHTS_FUSE1.3, INTERIOR_LIGHTS_FUSE1.4, INTERIOR_LIGHTS_FUSE1.5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: now also INTERIOR_LIGHTS_RELAY1.3; no longer INTERIOR_LIGHTS_RELAY1.1
- net at DASHBOARD_FUSE1.3, DASHBOARD_FUSE1.4, DASHBOARD_FUSE1.5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: now also DASHBOARD_RELAY1.3; no longer DASHBOARD_RELAY1.1
- net at D1.1, D2.1: now also DASHBOARD_RELAY1.4; no longer DASHBOARD_RELAY1.5
- net HAZARD_SWITCH_A: now reaches BMS_FUSE1.2
- net HAZARD_SWITCH_A: now also BMS_FUSE1.1, BMS_FUSE1.7, BMS_FUSE1.8, DASHBOARD_FUSE1.1, DASHBOARD_FUSE1.2, DASHBOARD_FUSE1.7, DASHBOARD_FUSE1.8, FLASHER_FUSE1.1, FLASHER_FUSE1.2, FLASHER_FUSE1.7, FLASHER_FUSE1.8, J1.1
- net at BMS_FUSE1.3, BMS_FUSE1.4, BMS_FUSE1.5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: no longer BMS_RELAY1.1
- net at D7.1, D8.1: now also BMS_RELAY1.4; no longer BMS_RELAY1.5
- net at HORN_FUSE1.3, HORN_FUSE1.4, HORN_FUSE1.5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: now also HORN_RELAY1.3; no longer HORN_RELAY1.1
- removed net BMS_GND: BMS_RELAY1.4, DASHBOARD_RELAY1.4, FWD_DRIVE_INHIBIT_RELAY1.4, HEADLIGHT_RELAY1.4, HIGHBEAM_RELAY1.4, HORN_RELAY1.4, IGNITION_RELAY1.4, INTERIOR_LIGHTS_RELAY1.4, LH_INDICATOR_RELAY1.4, REV_DRIVE_INHIBIT_RELAY1.4, RH_INDICATOR_RELAY1.4
- net LH_INDICATOR renamed LH_FRONT_INDICATOR
- net LH_FRONT_INDICATOR: now also LH_INDICATOR_RELAY1.1, J2.15, J3.3; no longer LH_INDICATOR_RELAY1.3
- net RH_INDICATOR renamed RH_FRONT_INDICATOR
- net RH_FRONT_INDICATOR: now also RH_INDICATOR_RELAY1.1, J2.16, J3.4; no longer RH_INDICATOR_RELAY1.3
- new net: RADIO_FUSE1.3, RADIO_FUSE1.4, RADIO_FUSE1.5, RADIO_FUSE1.6, RADIO_RELAY1.3
- new net: COOLANT_PUMP_FUSE1.3, COOLANT_PUMP_FUSE1.4, COOLANT_PUMP_FUSE1.5, COOLANT_PUMP_FUSE1.6, COOLANT_PUMP_RELAY1.3
- new net: COOLANT_PUMP_RELAY1.4, D3.1, D4.1
- new net BMS_FRONT_12V: BMS_RELAY1.1, J2.1, J3.1
- new net BMS_FRONT_GND: BMS_RELAY1.5, COOLANT_PUMP_RELAY1.5, DASHBOARD_RELAY1.5, DASHBOARD_RELAY2.5, FWD_DRIVE_INHIBIT_RELAY1.5, HEADLIGHT_RELAY1.5, HIGHBEAM_RELAY1.5, HORN_RELAY1.5, IGNITION_RELAY1.5, INTERIOR_LIGHTS_RELAY1.5, J2.19, J2.2, J2.4, J3.2, J4.3, LH_INDICATOR_RELAY1.5, RADIO_RELAY1.5, REV_DRIVE_INHIBIT_RELAY1.5, RH_INDICATOR_RELAY1.5
- new net BRAKE_SWITCH_B: J1.14, J2.5, J3.6
- new net CRUISE_SIGNAL: J1.21, J1.24
- new net DASHBOARD_5V: DASHBOARD_RELAY2.1, J4.7
- new net DASHBOARD_CHARGER_ON_SIGNAL: DASHBOARD_RELAY2.3, J4.8
- new net LH_HEADLIGHT: HEADLIGHT_RELAY1.1, J2.11, J2.12
Other:
- note added: "12v + gnd to shunt\n12v + gnd to negative contactor\ngnd to precharge and main contactors"
- note added: "BMS"
- note added: "CABIN"
- note added: "COOLANT PUMP"
- note added: "DASH"
- note added: "FRONT"
- note added: "Inverter\nTesla OBC\n\nStarted in drive mode and charge mode"
- note added: "REAR\n"
- note added: "SHIFTER"
- note added: "Turns on in drive mode and charge mode"
- note removed: "WATER PUMP"
- moved on the sheet: BMS_FUSE1, BMS_RELAY1, COOLANT_PUMP_FUSE1, D1, D10, D11, D12, D13, D14, D2, D7, D8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
