File: 12v-rear-pcb/12v-rear.kicad_sch (KiCad schematic)
At the start: 14 parts

Commit message: 12v rear backups
Parts:
- removed FRONT_1, FRONT_2, REAR_1, REAR_2: 282836-6, Socket:2828366, symbol Connector:282836-6
- removed LIM_FUSE1, REVERSE_LIGHT_FUSE1: 178.6165.0001, Socket:17861650001, symbol Connector:178.6165.0001
- removed LIM_RELAY1, REVERSE_LIGHT_RELAY1: DZ85AB-5-PCB, Socket:DZ85AB5PCB, symbol DZ85AB-5-PCB:DZ85AB-5-PCB
- added CHADEMO_FUSE: 178.6165.0001, Socket:17861650001, symbol Connector:178.6165.0001
- added CHADEMO_RELAY: DZ85AB-5-PCB, Socket:DZ85AB5PCB, symbol DZ85AB-5-PCB:DZ85AB-5-PCB
- added D2: 10A10, Diode_THT:DIOAD1165W56L425D185, symbol Diode:10A10
- added J1, J2, J3, J4, J5, J6, J7: 76825-0002, 768250002, symbol Connector:76825-0002
- added J10: 76825-0004, 768250004, symbol Connector:76825-0004
- renumbered TESLA_FUSE1 to CCS_FUSE1, TESLA_RELAY1 to CCS_RELAY1
Connections:
- net BMS_12V: now also J5.1
- net BMS_GND: now also J5.2
- net CHARGER_ON_SIGNAL: now also D2.1, J10.4
- net IGNITION_12V: now also J10.3
- net CHARGER_SWITCH_A renamed CCS_CHARGER_SWITCH_A
- net CCS_CHARGER_SWITCH_A: now also CHADEMO_FUSE.1, CHADEMO_FUSE.2, CHADEMO_FUSE.7, CHADEMO_FUSE.8, J10.1
- net CHARGER_SWITCH_B renamed CCS_CHARGER_SWITCH_B
- net GND renamed CCS_GND
- net CCS_GND: now also CHADEMO_RELAY.4, J10.2, J2.2, J3.2, J4.2, J6.2, J7.2
- net TESLA_12V renamed CCS_12V
- net CCS_12V: now also J2.1, J3.1, J6.1, J7.1
- new net: CHADEMO_FUSE.3, CHADEMO_FUSE.4, CHADEMO_FUSE.5, CHADEMO_FUSE.6, CHADEMO_RELAY.1
- new net CHADEMO_12V: CHADEMO_RELAY.3, J4.1
- new net CHADEMO_CHARGER_SWITCH_B: CHADEMO_RELAY.5, D2.2
- new net CHARGE_CONTACTORS_12V: J1.1
Other:
- note added: "BMS 12V supply"
- note added: "CCS Charging"
- note added: "CCS charge controller 12v supply"
- note added: "Chademo Charging"
- note added: "Chademo charge controller 12v supply"
- note added: "LIM 12V supply"
- note added: "LIM sense board 12V supply"
- note added: "Signals to/from front"
- note added: "Tesla 12V supply"
- note removed: "### Signals from front box which go directly to target ### * BRAKE_LIGHT * LH_REAR_INDICATOR * RH_REAR_INDICATOR * BMS 12V"
- note removed: "LIM"
- note removed: "REVERSE"
- note removed: "TESLA"
- moved on the sheet: CCS_FUSE1, CCS_RELAY1, D1
