File: dashboard-vcu/dashboard-vcu.kicad_sch (KiCad schematic)
At the start: 26 parts, among them IC2 TIP102, IC3 TIP102, J1 39300140, U1 Pico, U2 MCP2515-xSO, U3 SN65HVD230

Commit message: Dashboard vcu update
Parts:
- removed J1: 39300140, Connector:39300140, symbol Connector:39300140
- added X1: ATM13-12PB-12PC-BM03, ATM1312PB12PCBM03, symbol Connector:ATM13-12PB-12PC-BM03
Connections:
- net 12V: now also X1.B5
- net GND: now also C1.2, C2.2, PS1.1 (PGND), PS1.4 (AGND), R12.2, X1.B6
