File: 12v-lighting/12v-lighting.kicad_pcb (KiCad board)
At the start: 2 copper layers, 116.8 x 124.5 mm, 23 parts, among them J1 172065-0208, J2 172065-0208, J3 172065-0208, J4 172065-0208

Commit message: 12v lighting backups
Parts:
- removed INTERIOR_LIGHTS_FUSE1: 178.6165.0001, Connector:17861650001
- removed INTERIOR_LIGHTS_RELAY1: DZ85AB-5-PCB, Connector:DZ85AB5PCB
- added BRAKE_LIGHT_FUSE_1: 178.6165.0001, Socket:17861650001, F.Cu at (183.7, 117.7)
- added BRAKE_LIGHT_RELAY1: DZ85AB-5-PCB, Connector:DZ85AB5PCB, F.Cu at (205.0, 80.0)
- added CABIN_LIGHTS_FUSE1: 178.6165.0001, Socket:17861650001, F.Cu at (170.4, 117.7)
- added CABIN_LIGHTS_RELAY1: DZ85AB-5-PCB, Connector:DZ85AB5PCB, F.Cu at (170.0, 80.0)
- added J10: 76825-0002, Connector:768250002, F.Cu at (92.7, 48.3)
- added J11: 76825-0004, Connector:768250004, F.Cu at (200.2, 111.5)
- added J5: 76825-0002, Connector:768250002, F.Cu at (143.8, 112.2)
- added J6: 76825-0004, Connector:768250004, F.Cu at (122.4, 48.5)
- added J7: 76825-0004, Connector:768250004, F.Cu at (129.4, 112.1)
- added J8: 76825-0004, Connector:768250004, F.Cu at (271.3, 111.8)
- added J9: 76825-0004, Connector:768250004, F.Cu at (140.5, 48.5)
- added LIGHTING_IGNITION_RELAY1: DZ85AB-5-PCB, Connector:DZ85AB5PCB, F.Cu at (240.0, 80.0)
- added LIGHTING_MASTER_FUSE1: 178.6165.0001, Socket:17861650001, F.Cu at (219.0, 117.7)
- D10, D11, D12, D13, D14, D9: footprint Diode_THT:DIOAD1165W56L425D185 -> Diode_THT:D_DO-201AD_P15.24mm_Horizontal
- FLASHER_FUSE1, HEADLIGHT_FUSE1: footprint Connector:17861650001 -> Socket:17861650001
- J1, J2: value 172065-0208 -> 76825-0002; footprint Connector:1720650208 -> Connector:768250002
- J3, J4: value 172065-0208 -> 76825-0004; footprint Connector:1720650208 -> Connector:768250004
- moved H2 226.2 mm to (309.9, 42.2)
- moved H3 201.8 mm to (80.0, 119.1)
- moved HEADLIGHT_RELAY1 129.9 mm to (310.0, 80.0), turned to 180 degrees
- moved J4 128.6 mm to (295.0, 48.8), turned to 180 degrees
- moved LH_INDICATOR_RELAY1 122.5 mm to (135.0, 80.0), turned to 180 degrees
- moved RH_INDICATOR_RELAY1 101.1 mm to (100.0, 80.0), turned to 180 degrees
- moved J1 96.9 mm to (242.6, 111.7), turned to 0 degrees
- moved D9 92.7 mm to (100.8, 44.2), turned to -90 degrees
- moved H1 91.1 mm to (80.0, 40.9)
- moved D10 90.3 mm to (108.7, 44.2), turned to -90 degrees
- moved J3 90.2 mm to (275.5, 48.8)
- moved HIGHBEAM_RELAY1 83.5 mm to (275.0, 80.0), turned to 180 degrees
- moved G*** 70.3 mm to (240.3, 25.9)
- moved FLASHER_FUSE1 67.0 mm to (157.7, 117.7), turned to 90 degrees
- moved D13 66.1 mm to (91.7, 101.3), turned to -90 degrees
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Connections:
- D11 pad 2: LH_INDICATOR_SWITCH_B -> LH_INDICATOR_SWITCH_RETURN
- D12 pad 2: HAZARD_SWITCH_B -> HAZARD_SWITCH_RETURN
- D13 pad 2: RH_INDICATOR_SWITCH_B -> RH_INDICATOR_SWITCH_RETURN
- D14 pad 2: HAZARD_SWITCH_B -> HAZARD_SWITCH_RETURN
- FLASHER_FUSE1 pad 1: CABIN_PERM_12V -> 12V
- FLASHER_FUSE1 pad 2: CABIN_PERM_12V -> 12V
- FLASHER_FUSE1 pad 7: CABIN_PERM_12V -> 12V
- FLASHER_FUSE1 pad 8: CABIN_PERM_12V -> 12V
- HEADLIGHT_FUSE1 pad 1: BRAKE_SWITCH_A -> 12V
- HEADLIGHT_FUSE1 pad 2: BRAKE_SWITCH_A -> 12V
- HEADLIGHT_FUSE1 pad 7: BRAKE_SWITCH_A -> 12V
- HEADLIGHT_FUSE1 pad 8: BRAKE_SWITCH_A -> 12V
- HEADLIGHT_RELAY1 pad 1: HEADLIGHT -> LH_HEADLIGHT
- HEADLIGHT_RELAY1 pad 4: HEADLIGHT_SWITCH_B -> HEADLIGHT_SWITCH_RETURN
- HEADLIGHT_RELAY1 pad 5: GND -> LH_GND
- HIGHBEAM_RELAY1 pad 4: HIGHBEAM_SWITCH_B -> HIGHBEAM_SWITCH_RETURN
- HIGHBEAM_RELAY1 pad 5: GND -> LH_GND
- J1 pad 1: INTERIOR_LIGHTS -> LH_GND
- J1 pad 2: FLASHER_A -> 12V
- J2 pad 1: HAZARD_SWITCH_B -> BRAKE_SIGNAL_IN
- J2 pad 2: LH_INDICATOR_SWITCH_B -> IGNITION_ON_IN
- J3 pad 1: BRAKE_SWITCH_B -> LH_HEADLIGHT
- J3 pad 2: unconnected-(J3-Pad2) -> DASH_HIGHBEAM_INDICATOR
- J3 pad 4: FLASHER_B -> LH_GND
- J4 pad 1: DASH_HIGHBEAM_INDICATOR -> LH_HEADLIGHT
- J4 pad 2: HIGHBEAM_SWITCH_B -> DASH_HIGHBEAM_INDICATOR
- J4 pad 3: CABIN_PERM_12V -> LH_GND
- J4 pad 4: CABIN_PERM_12V -> unconnected-(J4-Pad4)
- LH_INDICATOR_RELAY1 pad 5: GND -> LH_GND
- RH_INDICATOR_RELAY1 pad 5: GND -> LH_GND
Routing:
- net LH_GND: track 0.00 -> 312.5 mm
- net GND: track 233.1 -> 0.00 mm
- net 12V: track 0.00 -> 215.2 mm
- net DASH_HIGHBEAM_INDICATOR: track 53.8 -> 184.2 mm
- net BRAKE_LIGHT: track 0.00 -> 100.1 mm
- net Net-(D11-Pad1): track 106.4 -> 25.6 mm
- net RH_INDICATOR_SWITCH_RETURN: track 0.00 -> 51.9 mm
- net LH_HEADLIGHT: track 0.00 -> 51.7 mm
- net HEADLIGHT_SWITCH_SEND: track 0.00 -> 48.7 mm
- net HEADLIGHT: track 45.0 -> 0.00 mm
- net Net-(CABIN_LIGHTS_FUSE1-Pad3): track 0.00 -> 43.4 mm
- net INTERIOR_LIGHT_SWITCH_B: track 43.3 -> 0.00 mm
- net CABIN_LIGHT_SWITCH_RETURN: track 0.00 -> 43.1 mm
- net HEADLIGHT_SWITCH_B: track 41.4 -> 0.00 mm
- net CABIN_PERM_12V: track 39.9 -> 0.00 mm
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Other:
- board size 116.8 x 124.5 mm -> 241 x 88 mm
- board text added: "BRAKE"
- board text added: "CABIN"
- board text added: "ELECTRIC MUSTANG Low voltage system - lighting Version 2"
- board text added: "HEALIGHT"
- board text added: "IGNITION"
- board text added: "J10 : front ind"
- board text added: "J1:12V"
- board text added: "J2:ignition"
- board text added: "J8:head/high sw"
- board text added: "LH IND"
- board text added: "LH headlight"
- board text added: "RH IND"
- board text added: "RH headlight"
- board text added: "brake"
- board text added: "cabin"
- board text added: "dash"
- board text added: "flasher"
- board text added: "headlight"
- board text added: "ind/haz sw"
- board text added: "main"
- board text added: "rear"
- board text removed: "ELECTRIC MUSTANG Low voltage system - lighting Version 1"
- board text removed: "FLASHER"
- board text removed: "HEADLIGHTS"
- board text removed: "INT LIGHTS"
- board text removed: "INTERIOR LIGHTS"
- board text removed: "LH INDICATOR"
- board text removed: "RH INDICATOR"

Commit message: lighting board. Add reverse light. Fix up a couple of issues.
Parts:
- added D1: 10A10, Diode_THT:D_DO-201AD_P15.24mm_Horizontal, F.Cu at (182.4, 49.4)
- added D2: 10A10, Diode_THT:D_DO-201AD_P15.24mm_Horizontal, F.Cu at (182.4, 56.1)
- added H5: MountingHole, MountingHole:MountingHole_3.2mm_M3, F.Cu at (143.5, 95.2)
- added H6: MountingHole, MountingHole:MountingHole_3.2mm_M3, F.Cu at (178.3, 63.5)
- added H7: MountingHole, MountingHole:MountingHole_3.2mm_M3, F.Cu at (213.6, 95.8)
- added H8: MountingHole, MountingHole:MountingHole_3.2mm_M3, F.Cu at (261.4, 61.0)
- added J12: 76825-0002, Library:768250002, F.Cu at (208.0, 48.6)
- added REVERSE_LIGHTS_FUSE1: 178.6165.0001, Library:17861650001, F.Cu at (252.5, 56.8)
- added REVERSE_LIGHT_RELAY1: DZ85AB-5-PCB, Library:DZ85AB5PCB, F.Cu at (222.6, 50.9)
- BRAKE_LIGHT_FUSE_1, CABIN_LIGHTS_FUSE1, FLASHER_FUSE1, HEADLIGHT_FUSE1, LIGHTING_MASTER_FUSE1: footprint Socket:17861650001 -> Library:17861650001
- BRAKE_LIGHT_RELAY1, CABIN_LIGHTS_RELAY1, HEADLIGHT_RELAY1, HIGHBEAM_RELAY1, LH_INDICATOR_RELAY1, LIGHTING_IGNITION_RELAY1, RH_INDICATOR_RELAY1: footprint Connector:DZ85AB5PCB -> Library:DZ85AB5PCB
- J1, J10, J2, J5: footprint Connector:768250002 -> Library:768250002
- J11, J3, J4, J6, J7, J8, J9: footprint Connector:768250004 -> Library:768250004
- moved G*** 95.0 mm to (295.9, 102.9)
- moved D13 2.42 mm to (89.3, 101.3)
- moved D11 2.42 mm to (112.3, 101.3)
- moved D12 2.42 mm to (104.5, 101.3)
- moved D14 2.42 mm to (96.9, 101.3)
- moved H1 1.48 mm to (80.8, 42.2)
- moved H3 1.27 mm to (81.0, 118.4)
- moved H4 1.05 mm to (309.1, 117.9)
Connections:
- net LH_GND renamed GND
- HEADLIGHT_FUSE1 pad 1: 12V -> HEADLIGHT_SWITCH_SEND
- HEADLIGHT_FUSE1 pad 2: 12V -> HEADLIGHT_SWITCH_SEND
- HEADLIGHT_FUSE1 pad 7: 12V -> HEADLIGHT_SWITCH_SEND
- HEADLIGHT_FUSE1 pad 8: 12V -> HEADLIGHT_SWITCH_SEND
Routing:
- net GND: track 312.5 -> 0.00 mm
- net LH_HEADLIGHT: track 51.7 -> 157.6 mm
- net TAIL_LIGHT: track 0.00 -> 72.6 mm
- net HEADLIGHT_SWITCH_SEND: track 48.7 -> 116.8 mm
- net DASH_HIGHBEAM_INDICATOR: track 184.2 -> 226.8 mm
- net 12V: track 215.2 -> 178.2 mm
- net REVERSE_SIGNAL: track 0.00 -> 27.7 mm
- net Net-(REVERSE_LIGHTS_FUSE1-Pad3): track 0.00 -> 26.7 mm
- net REVERSE_LIGHT: track 0.00 -> 18.1 mm
- net Net-(D11-Pad1): track 25.6 -> 32.3 mm
- net RH_FRONT_INDICATOR: track 73.4 -> 69.4 mm
- net Net-(HEADLIGHT_FUSE1-Pad3): track 37.4 -> 34.8 mm
- net Net-(LIGHTING_IGNITION_RELAY1-Pad3): track 35.7 -> 38.2 mm
- net HAZARD_SWITCH_RETURN: track 39.3 -> 40.7 mm
- net Net-(D13-Pad1): track 20.6 -> 21.5 mm
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- added copper zone on F.Cu, net 12V
- added copper zone on B.Cu, net GND
Other:
- board text added: "ELECTRIC MUSTANG Low voltage system - lighting Version 2 ©2023"
- board text added: "FLASHER"
- board text added: "J1 : 12V IN"
- board text added: "J10 : FRONT IND"
- board text added: "J11 : CABIN"
- board text added: "J12 : REVERSE"
- board text added: "J3 : LH HL"
- board text added: "J4 : RH HL"
- board text added: "J5 : FLASHER"
- board text added: "J6 : REAR"
- board text added: "J7 : IND/HAZ SW"
- board text added: "J8 : HL/HB SW"
- board text added: "J9 : DASH"
- board text added: "REVERSE"
- board text removed: "ELECTRIC MUSTANG Low voltage system - lighting Version 2"
- board text removed: "J10 : front ind"
- board text removed: "J1:12V"
- board text removed: "J8:head/high sw"
- board text removed: "LH headlight"
- board text removed: "RH headlight"
- board text removed: "brake"
- board text removed: "cabin"
- board text removed: "dash"
- board text removed: "flasher"
- board text removed: "ind/haz sw"
- board text removed: "main"
- board text removed: "rear"
