File: 12v-lighting/12v-lighting.kicad_sch (KiCad schematic)
At the start: 22 parts, among them J1 172065-0208, J2 172065-0208, J3 172065-0208, J4 172065-0208

Commit message: 12v lighting backups
Parts:
- removed J1, J2, J3, J4: 172065-0208, 1720650208, symbol Connector:172065-0208
- added BRAKE_LIGHT_FUSE_1, LIGHTING_MASTER_FUSE1: 178.6165.0001, Socket:17861650001, symbol Connector:178.6165.0001
- added BRAKE_LIGHT_RELAY1, LIGHTING_IGNITION_RELAY1: DZ85AB-5-PCB, Connector:DZ85AB5PCB, symbol DZ85AB-5-PCB:DZ85AB-5-PCB
- added J1, J10, J2, J5: 76825-0002, 768250002, symbol Connector:76825-0002
- added J11, J3, J4, J6, J7, J8, J9: 76825-0004, 768250004, symbol Connector:76825-0004
- CABIN_LIGHTS_FUSE1: renamed from INTERIOR_LIGHTS_FUSE1; footprint Connector:17861650001 -> Socket:17861650001
- D10, D11, D12, D13, D14, D9: footprint Diode_THT:DIOAD1165W56L425D185 -> Diode_THT:D_DO-201AD_P15.24mm_Horizontal
- FLASHER_FUSE1, HEADLIGHT_FUSE1: footprint Connector:17861650001 -> Socket:17861650001
- renumbered INTERIOR_LIGHTS_RELAY1 to CABIN_LIGHTS_RELAY1
Connections:
- net CABIN_PERM_12V is gone; now on net 12V: CABIN_LIGHTS_FUSE1.1, CABIN_LIGHTS_FUSE1.2, CABIN_LIGHTS_FUSE1.7, CABIN_LIGHTS_FUSE1.8, FLASHER_FUSE1.1, FLASHER_FUSE1.2, FLASHER_FUSE1.7, FLASHER_FUSE1.8
- net DASH_HIGHBEAM_INDICATOR: now also J3.2, J4.2, J9.2
- net DASH_INDICATOR_INDICATOR: now also J9.4
- net FLASHER_A: now also J5.1
- net FLASHER_B: now also J5.2
- net GND: now also BRAKE_LIGHT_RELAY1.5, J1.1, J3.4, J4.3, J9.1, LIGHTING_IGNITION_RELAY1.5
- net LH_FRONT_INDICATOR: now also J10.1, J6.1
- net RH_FRONT_INDICATOR: now also J10.2, J6.2
- net BRAKE_SWITCH_A renamed 12V
- net 12V: now also BRAKE_LIGHT_FUSE_1.1, BRAKE_LIGHT_FUSE_1.2, BRAKE_LIGHT_FUSE_1.7, BRAKE_LIGHT_FUSE_1.8, J1.2, J11.2, J7.4, LIGHTING_MASTER_FUSE1.1, LIGHTING_MASTER_FUSE1.2, LIGHTING_MASTER_FUSE1.7, LIGHTING_MASTER_FUSE1.8
- net HAZARD_SWITCH_B renamed HAZARD_SWITCH_RETURN
- net HAZARD_SWITCH_RETURN: now also J7.3
- net HEADLIGHT renamed LH_HEADLIGHT
- net LH_HEADLIGHT: now also J3.1, J4.1
- net HEADLIGHT_SWITCH_B renamed HEADLIGHT_SWITCH_RETURN
- net HEADLIGHT_SWITCH_RETURN: now also J8.2
- net HIGHBEAM_SWITCH_B renamed HIGHBEAM_SWITCH_RETURN
- net HIGHBEAM_SWITCH_RETURN: now also J8.1
- net INTERIOR_LIGHTS renamed CABIN_LIGHT
- net CABIN_LIGHT: now also J11.1
- net INTERIOR_LIGHT_SWITCH_B renamed CABIN_LIGHT_SWITCH_RETURN
- net CABIN_LIGHT_SWITCH_RETURN: now also J11.3
- net LH_INDICATOR_SWITCH_B renamed LH_INDICATOR_SWITCH_RETURN
- net LH_INDICATOR_SWITCH_RETURN: now also J7.1
- net RH_INDICATOR_SWITCH_B renamed RH_INDICATOR_SWITCH_RETURN
- net RH_INDICATOR_SWITCH_RETURN: now also J7.2
- new net: BRAKE_LIGHT_FUSE_1.3, BRAKE_LIGHT_FUSE_1.4, BRAKE_LIGHT_FUSE_1.5, BRAKE_LIGHT_FUSE_1.6, BRAKE_LIGHT_RELAY1.3
- new net: LIGHTING_IGNITION_RELAY1.3, LIGHTING_MASTER_FUSE1.3, LIGHTING_MASTER_FUSE1.4, LIGHTING_MASTER_FUSE1.5, LIGHTING_MASTER_FUSE1.6
- new net BRAKE_LIGHT: BRAKE_LIGHT_RELAY1.1, J6.4
- new net BRAKE_SIGNAL_IN: BRAKE_LIGHT_RELAY1.4, J2.1
- new net HEADLIGHT_SWITCH_SEND: J8.3, J8.4, LIGHTING_IGNITION_RELAY1.1
- new net IGNITION_ON_IN: J2.2, LIGHTING_IGNITION_RELAY1.4
- new net TAIL_LIGHT: J6.3
Other:
- note added: "12V Batt"
- note added: "12v-front"
- note added: "BRAKE LIGHT"
- note added: "CABIN LIGHTS"
- note added: "HEADLIGHT/HIGHBEAM"
- note added: "IGNITION Separate permanent feed from 12V battery comes into this board. Battery power is switched by the ignition signal from the 12v-front board."
- note added: "LH front lights"
- note added: "RH front lights"
- note added: "cabin"
- note added: "dash"
- note added: "flasher"
- note added: "front indicators"
- note added: "indicator/hazard controls"
- note added: "lighting switches"
- note added: "rear"
- note removed: "HEADLIGHT"
- note removed: "INTERIOR LIGHTS"
- moved on the sheet: CABIN_LIGHTS_FUSE1, CABIN_LIGHTS_RELAY1, D10, D11, D12, D13, D14, D9, FLASHER_FUSE1, HEADLIGHT_FUSE1, HEADLIGHT_RELAY1, HIGHBEAM_RELAY1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

Commit message: lighting board. Add reverse light. Fix up a couple of issues.
Parts:
- added D1, D2: 10A10, Diode_THT:D_DO-201AD_P15.24mm_Horizontal, symbol Diode:10A10
- added H5, H6, H7, H8: MountingHole, MountingHole:MountingHole_3.2mm_M3, symbol Mechanical:MountingHole
- added J12: 76825-0002, 768250002, symbol Connector:76825-0002
- added REVERSE_LIGHTS_FUSE1: 178.6165.0001, Library:17861650001, symbol Connector:178.6165.0001
- added REVERSE_LIGHT_RELAY1: DZ85AB-5-PCB, Library:DZ85AB5PCB, symbol DZ85AB-5-PCB:DZ85AB-5-PCB
- BRAKE_LIGHT_FUSE_1, CABIN_LIGHTS_FUSE1, FLASHER_FUSE1, HEADLIGHT_FUSE1, LIGHTING_MASTER_FUSE1: footprint Socket:17861650001 -> Library:17861650001
- BRAKE_LIGHT_RELAY1, CABIN_LIGHTS_RELAY1, HEADLIGHT_RELAY1, HIGHBEAM_RELAY1, LH_INDICATOR_RELAY1, LIGHTING_IGNITION_RELAY1, RH_INDICATOR_RELAY1: footprint Connector:DZ85AB5PCB -> Library:DZ85AB5PCB
Connections:
- net 12V: no longer HEADLIGHT_FUSE1.1, HEADLIGHT_FUSE1.2, HEADLIGHT_FUSE1.7, HEADLIGHT_FUSE1.8
- net DASH_HIGHBEAM_INDICATOR: now also D2.2
- net GND: now also REVERSE_LIGHT_RELAY1.5
- net HEADLIGHT_SWITCH_SEND: now also HEADLIGHT_FUSE1.1, HEADLIGHT_FUSE1.2, HEADLIGHT_FUSE1.7, HEADLIGHT_FUSE1.8, REVERSE_LIGHTS_FUSE1.1, REVERSE_LIGHTS_FUSE1.2, REVERSE_LIGHTS_FUSE1.7, REVERSE_LIGHTS_FUSE1.8
- net LH_HEADLIGHT: now also D1.2
- net TAIL_LIGHT: now also D1.1, D2.1
- new net: REVERSE_LIGHTS_FUSE1.3, REVERSE_LIGHTS_FUSE1.4, REVERSE_LIGHTS_FUSE1.5, REVERSE_LIGHTS_FUSE1.6, REVERSE_LIGHT_RELAY1.3
- new net REVERSE_LIGHT: J12.1, REVERSE_LIGHT_RELAY1.1
- new net REVERSE_SIGNAL: J12.2, REVERSE_LIGHT_RELAY1.4
Other:
- note added: "REVERSE LIGHT"
- moved on the sheet: H1, H2, H3, H4, HEADLIGHT_FUSE1, HEADLIGHT_RELAY1, HIGHBEAM_RELAY1
